File: USB_IF.sch (KiCad schematic (older format))
At the start: 9 parts

Commit message: Started adding component values and tidying up
Parts:
- C?: value C -> 100n
- C?: value CP -> 10u
Connections:
- no-connect marks 0 -> 14
Changed lines of the file:
@@
 P 3150 1750
 F 0 "C?" H 3175 1850 50  0000 L CNN
-F 1 "C" H 3175 1650 50  0000 L CNN
+F 1 "100n" H 3175 1650 50  0000 L CNN
 F 2 "" H 3188 1600 30  0000 C CNN
 F 3 "" H 3150 1750 60  0000 C CNN
@@
 P 3500 1750
 F 0 "C?" H 3525 1850 50  0000 L CNN
-F 1 "CP" H 3525 1650 50  0000 L CNN
+F 1 "10u" H 3525 1650 50  0000 L CNN
 F 2 "" H 3538 1600 30  0000 C CNN
 F 3 "" H 3500 1750 60  0000 C CNN
@@
 Wire Wire Line
 	2700 4600 2950 4600
+NoConn ~ 5150 3100
+NoConn ~ 5150 3250
+NoConn ~ 5150 3400
+NoConn ~ 5150 3550
+NoConn ~ 5150 3700
+NoConn ~ 5150 3850
+NoConn ~ 5150 4300
+NoConn ~ 5150 4450
+NoConn ~ 5150 4600
+NoConn ~ 2950 4150
+NoConn ~ 2950 4000
+NoConn ~ 2950 3700
+NoConn ~ 1600 2400
+NoConn ~ 1300 2000
 $EndSCHEMATC

Commit message: added component values and most packages. Still missing micro usb
Parts:
- C1, C2: renamed from C?; footprint (none) -> Resistors_SMD:R_0805_HandSoldering
- D1, D2: renamed from D?; footprint (none) -> Resistors_SMD:R_0805_HandSoldering
- R1, R2, R3: renamed from R?; footprint (none) -> Resistors_SMD:R_0805_HandSoldering
- U1: renamed from U?; footprint (none) -> Housings_SSOP:SSOP-28_5.3x10.2mm_Pitch0.65mm
- gave numbers to parts that had none: 1
Changed lines of the file:
@@
 $EndDescr
 $Comp
-L FT232RL U?
+L FT232RL U1
 U 1 1 563FE286
 P 4050 3700
-F 0 "U?" H 3300 4900 60  0000 C CNN
+F 0 "U1" H 3300 4900 60  0000 C CNN
 F 1 "FT232RL" H 4050 3700 60  0000 C CNN
-F 2 "" H 4050 3700 60  0000 C CNN
+F 2 "Housings_SSOP:SSOP-28_5.3x10.2mm_Pitch0.65mm" H 4050 3700 60  0001 C CNN
 F 3 "" H 4050 3700 60  0000 C CNN
 	1    4050 3700
@@
 $EndComp
 $Comp
-L C C?
+L C C1
 U 1 1 563FE2C9
 P 3150 1750
-F 0 "C?" H 3175 1850 50  0000 L CNN
+F 0 "C1" H 3175 1850 50  0000 L CNN
 F 1 "100n" H 3175 1650 50  0000 L CNN
-F 2 "" H 3188 1600 30  0000 C CNN
+F 2 "Resistors_SMD:R_0805_HandSoldering" H 3188 1600 30  0001 C CNN
 F 3 "" H 3150 1750 60  0000 C CNN
 	1    3150 1750
@@
 $EndComp
 $Comp
-L CP C?
+L CP C2
 U 1 1 563FE30A
 P 3500 1750
-F 0 "C?" H 3525 1850 50  0000 L CNN
+F 0 "C2" H 3525 1850 50  0000 L CNN
 F 1 "10u" H 3525 1650 50  0000 L CNN
-F 2 "" H 3538 1600 30  0000 C CNN
+F 2 "Resistors_SMD:R_0805_HandSoldering" H 3538 1600 30  0001 C CNN
 F 3 "" H 3500 1750 60  0000 C CNN
 	1    3500 1750
@@
 $EndComp
 $Comp
-L R R?
+L R R3
 U 1 1 563FE3C3
 P 6900 2950
-F 0 "R?" V 6980 2950 50  0000 C CNN
+F 0 "R3" V 6980 2950 50  0000 C CNN
 F 1 "1k" V 6900 2950 50  0000 C CNN
-F 2 "" V 6830 2950 30  0000 C CNN
+F 2 "Resistors_SMD:R_0805_HandSoldering" V 6830 2950 30  0001 C CNN
 F 3 "" H 6900 2950 30  0000 C CNN
 	1    6900 2950
@@
 $EndComp
 $Comp
-L USB_OTG P?
+L USB_OTG P1
 U 1 1 563FE402
 P 1700 2100
-F 0 "P?" H 2025 1975 50  0000 C CNN
+F 0 "P1" H 2025 1975 50  0000 C CNN
 F 1 "USB_OTG" H 1700 2300 50  0000 C CNN
-F 2 "" V 1650 2000 60  0000 C CNN
+F 2 "" V 1650 2000 60  0001 C CNN
 F 3 "" V 1650 2000 60  0000 C CNN
 	1    1700 2100
@@
 Connection ~ 4050 5200
 $Comp
-L GNDPWR #PWR?
+L GNDPWR #PWR01
 U 1 1 563FE6D9
 P 3900 5400
-F 0 "#PWR?" H 3900 5200 50  0001 C CNN
+F 0 "#PWR01" H 3900 5200 50  0001 C CNN
 F 1 "GNDPWR" H 3900 5270 50  0000 C CNN
 F 2 "" H 3900 5350 60  0000 C CNN
@@
 $EndComp
 $Comp
-L +5V #PWR?
+L +5V #PWR02
 U 1 1 563FE720
 P 2300 2800
-F 0 "#PWR?" H 2300 2650 50  0001 C CNN
+F 0 "#PWR02" H 2300 2650 50  0001 C CNN
 F 1 "+5V" H 2300 2940 50  0000 C CNN
 F 2 "" H 2300 2800 60  0000 C CNN
@@
 Connection ~ 3900 5200
 $Comp
-L GNDPWR #PWR?
+L GNDPWR #PWR03
 U 1 1 563FE7A1
 P 1500 2550
-F 0 "#PWR?" H 1500 2350 50  0001 C CNN
+F 0 "#PWR03" H 1500 2350 50  0001 C CNN
 F 1 "GNDPWR" H 1500 2420 50  0000 C CNN
 F 2 "" H 1500 2500 60  0000 C CNN
@@
 	1500 2400 1500 2550
 $Comp
-L GNDPWR #PWR?
+L GNDPWR #PWR04
 U 1 1 563FE975
 P 3300 2100
-F 0 "#PWR?" H 3300 1900 50  0001 C CNN
+F 0 "#PWR04" H 3300 1900 50  0001 C CNN
 F 1 "GNDPWR" H 3300 1970 50  0000 C CNN
 F 2 "" H 3300 2050 60  0000 C CNN
@@
 $EndComp
 $Comp
-L +5V #PWR?
+L +5V #PWR05
 U 1 1 563FE997
 P 3300 1400
-F 0 "#PWR?" H 3300 1250 50  0001 C CNN
+F 0 "#PWR05" H 3300 1250 50  0001 C CNN
 F 1 "+5V" H 3300 1540 50  0000 C CNN
 F 2 "" H 3300 1400 60  0000 C CNN
@@
 	3150 1900 3150 2000
 $Comp
-L LED D?
+L LED D2
 U 1 1 563FEAD6
 P 6900 3450
-F 0 "D?" H 6900 3550 50  0000 C CNN
+F 0 "D2" H 6900 3550 50  0000 C CNN
 F 1 "LED" H 6900 3350 50  0000 C CNN
-F 2 "" H 6900 3450 60  0000 C CNN
+F 2 "Resistors_SMD:R_0805_HandSoldering" H 6900 3450 60  0001 C CNN
 F 3 "" H 6900 3450 60  0000 C CNN
 	1    6900 3450
@@
 $EndComp
 $Comp
-L LED D?
+L LED D1
 U 1 1 563FEE17
 P 6550 3450
-F 0 "D?" H 6550 3550 50  0000 C CNN
+F 0 "D1" H 6550 3550 50  0000 C CNN
 F 1 "LED" H 6550 3350 50  0000 C CNN
-F 2 "" H 6550 3450 60  0000 C CNN
+F 2 "Resistors_SMD:R_0805_HandSoldering" H 6550 3450 60  0001 C CNN
 F 3 "" H 6550 3450 60  0000 C CNN
 	1    6550 3450
@@
 	6900 3650 6900 4150
 $Comp
-L R R?
+L R R2
 U 1 1 563FEF80
 P 6550 2950
-F 0 "R?" V 6630 2950 50  0000 C CNN
+F 0 "R2" V 6630 2950 50  0000 C CNN
 F 1 "1k" V 6550 2950 50  0000 C CNN
-F 2 "" V 6480 2950 30  0000 C CNN
+F 2 "Resistors_SMD:R_0805_HandSoldering" V 6480 2950 30  0001 C CNN
 F 3 "" H 6550 2950 30  0000 C CNN
 	1    6550 2950
@@
 	6900 3250 6900 3100
 $Comp
-L +5V #PWR?
+L +5V #PWR06
 U 1 1 563FF179
 P 6550 2700
-F 0 "#PWR?" H 6550 2550 50  0001 C CNN
+F 0 "#PWR06" H 6550 2550 50  0001 C CNN
 F 1 "+5V" H 6550 2840 50  0000 C CNN
 F 2 "" H 6550 2700 60  0000 C CNN
@@
 $EndComp
 $Comp
-L +5V #PWR?
+L +5V #PWR07
 U 1 1 563FF1A1
 P 6900 2700
-F 0 "#PWR?" H 6900 2550 50  0001 C CNN
+F 0 "#PWR07" H 6900 2550 50  0001 C CNN
 F 1 "+5V" H 6900 2840 50  0000 C CNN
 F 2 "" H 6900 2700 60  0000 C CNN
@@
 FTDI_IN_RXD
 $Comp
-L R R?
+L R R1
 U 1 1 563FF62A
 P 5350 2800
-F 0 "R?" V 5430 2800 50  0000 C CNN
+F 0 "R1" V 5430 2800 50  0000 C CNN
 F 1 "10R" V 5350 2800 50  0000 C CNN
-F 2 "" V 5280 2800 30  0000 C CNN
+F 2 "Resistors_SMD:R_0805_HandSoldering" V 5280 2800 30  0001 C CNN
 F 3 "" H 5350 2800 30  0000 C CNN
 	1    5350 2800

Commit message: Added a USB socket with GND set as a power output to pass DRC, and gave a first stab at a placement. Man that's tight! Components both side required??
Parts:
- C1: footprint Resistors_SMD:R_0805_HandSoldering -> Resistors_SMD:R_0603_HandSoldering
- P1: footprint (none) -> ab2_usb:AB2_USB_MICRO_SMD
Changed lines of the file:
@@
 F 0 "C1" H 3175 1850 50  0000 L CNN
 F 1 "100n" H 3175 1650 50  0000 L CNN
-F 2 "Resistors_SMD:R_0805_HandSoldering" H 3188 1600 30  0001 C CNN
+F 2 "Resistors_SMD:R_0603_HandSoldering" H 3188 1600 30  0001 C CNN
 F 3 "" H 3150 1750 60  0000 C CNN
 	1    3150 1750
@@
 F 0 "P1" H 2025 1975 50  0000 C CNN
 F 1 "USB_OTG" H 1700 2300 50  0000 C CNN
-F 2 "" V 1650 2000 60  0001 C CNN
+F 2 "ab2_usb:AB2_USB_MICRO_SMD" V 1650 2000 60  0001 C CNN
 F 3 "" V 1650 2000 60  0000 C CNN
 	1    1700 2100

Commit message: Dodgy layout added, etc
Parts:
- P1: footprint ab2_usb:AB2_USB_MICRO_SMD -> Connect:USB_Micro-B; symbol USB_OTG -> USB_OTG-RESCUE-weatherstation
Changed lines of the file:
@@
 EESchema Schematic File Version 2
+LIBS:weatherstation-rescue
 LIBS:power
 LIBS:device
@@
 $EndComp
 $Comp
-L USB_OTG P1
+L USB_OTG-RESCUE-weatherstation P1
 U 1 1 563FE402
 P 1700 2100
 F 0 "P1" H 2025 1975 50  0000 C CNN
 F 1 "USB_OTG" H 1700 2300 50  0000 C CNN
-F 2 "ab2_usb:AB2_USB_MICRO_SMD" V 1650 2000 60  0001 C CNN
+F 2 "Connect:USB_Micro-B" V 1650 2000 60  0001 C CNN
 F 3 "" V 1650 2000 60  0000 C CNN
 	1    1700 2100

Commit message: Added some RS part numbers for switches and usb
Parts:
- P1: RS_Part (none) -> http://uk.rs-online.com/web/p/micro-usb-connectors/7795106/
Changed lines of the file:
@@
 EESchema Schematic File Version 2
-LIBS:weatherstation-rescue
 LIBS:power
 LIBS:device
@@
 F 2 "Connect:USB_Micro-B" V 1650 2000 60  0001 C CNN
 F 3 "" V 1650 2000 60  0000 C CNN
+F 4 "http://uk.rs-online.com/web/p/micro-usb-connectors/7795106/" H 1700 2100 60  0001 C CNN "RS_Part"
 	1    1700 2100
 	-1   0    0    -1
