File: display.sch (KiCad schematic (older format))
At the start: 1 part, among them P2 CONN_01X08

Commit message: Added logo, sensor, manufacturing data'
Parts:
- added IC1: TMP100, SOT-23-6, symbol TMP100
Connections:
- net +5V: now also IC1.4 (VCC)
- net DISP_SCL: now also IC1.1 (SCL)
- net DISP_SDA: now also IC1.6 (SDA)
- net GNDPWR: now also IC1.2 (GND), IC1.3 (A1)
- no-connect marks 3 -> 6
Changed lines of the file:
@@
 $EndComp
 $Comp
-L +5V #PWR024
+L +5V #PWR26
 U 1 1 56403310
 P 4250 3250
-F 0 "#PWR024" H 4250 3100 50  0001 C CNN
+F 0 "#PWR26" H 4250 3100 50  0001 C CNN
 F 1 "+5V" H 4250 3390 50  0000 C CNN
 F 2 "" H 4250 3250 60  0000 C CNN
@@
 $EndComp
 $Comp
-L GNDPWR #PWR025
+L GNDPWR #PWR27
 U 1 1 56403326
 P 4500 3600
-F 0 "#PWR025" H 4500 3400 50  0001 C CNN
+F 0 "#PWR27" H 4500 3400 50  0001 C CNN
 F 1 "GNDPWR" H 4500 3470 50  0000 C CNN
 F 2 "" H 4500 3550 60  0000 C CNN
@@
 SDA
 Wire Wire Line
-	4650 2700 4400 2700
+	4050 2700 4650 2700
 Wire Wire Line
-	4650 2800 4400 2800
+	3900 2800 4650 2800
 Text HLabel 5950 2100 0    60   3State ~ 0
 DISP_SCL
@@
 Text Notes 5600 3000 0    60   ~ 0
 Note, pullups are fitted on display module, 10k to 3V3
+$Comp
+L TMP100 IC1
+U 1 1 5649DE51
+P 3050 2850
+F 0 "IC1" H 2850 3100 40  0000 C CNN
+F 1 "TMP100" H 3350 2550 40  0000 C CNN
+F 2 "SOT-23-6" H 3050 2850 35  0000 C CIN
+F 3 "" H 3050 2850 60  0000 C CNN
+	1    3050 2850
+	1    0    0    -1
+$EndComp
+$Comp
+L GNDPWR #PWR24
+U 1 1 5649DFB4
+P 2500 3250
+F 0 "#PWR24" H 2500 3050 50  0001 C CNN
+F 1 "GNDPWR" H 2500 3120 50  0000 C CNN
+F 2 "" H 2500 3200 60  0000 C CNN
+F 3 "" H 2500 3200 60  0000 C CNN
+	1    2500 3250
+	1    0    0    -1
+$EndComp
+Wire Wire Line
+	2650 3050 2500 3050
+Wire Wire Line
+	2500 3050 2500 3250
+Wire Wire Line
+	3050 3250 2800 3250
+Wire Wire Line
+	2800 3250 2800 3200
+Wire Wire Line
+	2800 3200 2500 3200
+Connection ~ 2500 3200
+Wire Wire Line
+	3450 2750 4050 2750
+Wire Wire Line
+	4050 2750 4050 2700
+Wire Wire Line
+	3900 2800 3900 2900
+Wire Wire Line
+	3900 2900 3450 2900
+$Comp
+L +5V #PWR25
+U 1 1 5649E01D
+P 3050 2400
+F 0 "#PWR25" H 3050 2250 50  0001 C CNN
+F 1 "+5V" H 3050 2540 50  0000 C CNN
+F 2 "" H 3050 2400 60  0000 C CNN
+F 3 "" H 3050 2400 60  0000 C CNN
+	1    3050 2400
+	1    0    0    -1
+$EndComp
+Wire Wire Line
+	3050 2400 3050 2500
+NoConn ~ 2650 2900
+NoConn ~ 4400 3900
+NoConn ~ 2950 2750
 $EndSCHEMATC
